File: 20-12-2016/EB_DRV/Batterry_Measurment.sch (KiCad schematic (older format))
At the start: 3 parts, among them P13 CONN_01X02

Commit message: Added_footprints(not all)
Parts:
- P13: footprint (none) -> Pin_Headers:Pin_Header_Straight_1x02_Pitch2.54mm
- R65, R66: footprint (none) -> Resistors_SMD:R_0805_HandSoldering
Changed lines of the file:
@@
 F 0 "R65" V 5080 2350 50  0000 C CNN
 F 1 "R" V 5000 2350 50  0000 C CNN
-F 2 "" V 4930 2350 50  0000 C CNN
+F 2 "Resistors_SMD:R_0805_HandSoldering" V 4930 2350 50  0001 C CNN
 F 3 "" H 5000 2350 50  0000 C CNN
 	1    5000 2350
@@
 F 0 "R66" V 5080 2850 50  0000 C CNN
 F 1 "R" V 5000 2850 50  0000 C CNN
-F 2 "" V 4930 2850 50  0000 C CNN
+F 2 "Resistors_SMD:R_0805_HandSoldering" V 4930 2850 50  0001 C CNN
 F 3 "" H 5000 2850 50  0000 C CNN
 	1    5000 2850
@@
 U 1 1 585A8883
 P 5000 4150
+AR Path="/585A8883" Ref="P13"  Part="1"
+AR Path="/585445EE/585A8883" Ref="P13"  Part="1"
 F 0 "P13" H 5000 4300 50  0000 C CNN
 F 1 "CONN_01X02" V 5100 4150 50  0000 C CNN
-F 2 "" H 5000 4150 50  0000 C CNN
+F 2 "Pin_Headers:Pin_Header_Straight_1x02_Pitch2.54mm" H 5000 4150 50  0001 C CNN
 F 3 "" H 5000 4150 50  0000 C CNN
 	1    5000 4150
