File: 20-12-2016/EB_DRV/Bike_sensors.sch (KiCad schematic (older format))
At the start: 8 parts, among them P10 F_BREAK_CONN, P11 R_BREAK_CONN, P14 R_BREAK_CONN

Commit message: Added_footprints(not all)
Parts:
- P10, P11, P14: footprint (none) -> Pin_Headers:Pin_Header_Straight_1x03_Pitch2.54mm
Changed lines of the file:
@@
 F 0 "P10" H 4800 2450 50  0000 C CNN
 F 1 "F_BREAK_CONN" V 4900 2250 50  0000 C CNN
-F 2 "" H 4800 2250 50  0000 C CNN
+F 2 "Pin_Headers:Pin_Header_Straight_1x03_Pitch2.54mm" H 4800 2250 50  0001 C CNN
 F 3 "" H 4800 2250 50  0000 C CNN
 	1    4800 2250
@@
 F 0 "P11" H 4850 3750 50  0000 C CNN
 F 1 "R_BREAK_CONN" V 4950 3550 50  0000 C CNN
-F 2 "" H 4850 3550 50  0000 C CNN
+F 2 "Pin_Headers:Pin_Header_Straight_1x03_Pitch2.54mm" H 4850 3550 50  0001 C CNN
 F 3 "" H 4850 3550 50  0000 C CNN
 	1    4850 3550
@@
 F 0 "P14" H 4850 4700 50  0000 C CNN
 F 1 "R_BREAK_CONN" V 4950 4500 50  0000 C CNN
-F 2 "" H 4850 4500 50  0000 C CNN
+F 2 "Pin_Headers:Pin_Header_Straight_1x03_Pitch2.54mm" H 4850 4500 50  0001 C CNN
 F 3 "" H 4850 4500 50  0000 C CNN
 	1    4850 4500
