File: 20-12-2016/EB_DRV/EB_DRV.sch (KiCad schematic (older format))
At the start: 23 parts, among them P1 HALL/Encoder, P15 light debug, P2 LIghts_Connector, P3 Battery_Charger_Output, P4 DEBUG_CON, P5 BT_CON, P6 PROG_CON_1, P7 PROG_CON_2, U1 MINi_USB_JACK

Commit message: Added_footprints(not all)
Parts:
- D1, D2, D3: footprint (none) -> LEDs:LED_0805
- P1, P5: footprint (none) -> Pin_Headers:Pin_Header_Straight_1x06_Pitch2.54mm
- P15, P3, P4: footprint (none) -> Pin_Headers:Pin_Header_Straight_1x02_Pitch2.54mm
- P2: footprint (none) -> Pin_Headers:Pin_Header_Straight_1x10_Pitch2.54mm
- P6, P7: footprint (none) -> Pin_Headers:Pin_Header_Straight_1x05_Pitch2.54mm
- R3: footprint (none) -> Resistors_SMD:R_0805_HandSoldering
Changed lines of the file:
@@
 F 0 "P1" H 1050 7350 50  0000 C CNN
 F 1 "HALL/Encoder" V 1150 7000 50  0000 C CNN
-F 2 "" H 1050 7000 50  0000 C CNN
+F 2 "Pin_Headers:Pin_Header_Straight_1x06_Pitch2.54mm" H 1050 7000 50  0001 C CNN
 F 3 "" H 1050 7000 50  0000 C CNN
 	1    1050 7000
@@
 F 0 "P5" H 3950 3850 50  0000 C CNN
 F 1 "BT_CON" V 4050 3500 50  0000 C CNN
-F 2 "" H 3950 3500 50  0000 C CNN
+F 2 "Pin_Headers:Pin_Header_Straight_1x06_Pitch2.54mm" H 3950 3500 50  0001 C CNN
 F 3 "" H 3950 3500 50  0000 C CNN
 	1    3950 3500
@@
 F 0 "D1" H 7600 5875 50  0000 L CNN
 F 1 "Led_Small" H 7475 5650 50  0000 L CNN
-F 2 "" V 7650 5750 50  0000 C CNN
+F 2 "LEDs:LED_0805" V 7650 5750 50  0001 C CNN
 F 3 "" V 7650 5750 50  0000 C CNN
 	1    7650 5750
@@
 F 0 "D2" H 8000 5875 50  0000 L CNN
 F 1 "Led_Small" H 7875 5650 50  0000 L CNN
-F 2 "" V 8050 5750 50  0000 C CNN
+F 2 "LEDs:LED_0805" V 8050 5750 50  0001 C CNN
 F 3 "" V 8050 5750 50  0000 C CNN
 	1    8050 5750
@@
 F 0 "D3" H 8250 5875 50  0000 L CNN
 F 1 "Led_Small" H 8125 5650 50  0000 L CNN
-F 2 "" V 8300 5750 50  0000 C CNN
+F 2 "LEDs:LED_0805" V 8300 5750 50  0001 C CNN
 F 3 "" V 8300 5750 50  0000 C CNN
 	1    8300 5750
@@
 F 0 "P6" H 3950 4450 50  0000 C CNN
 F 1 "PROG_CON_1" V 4050 4150 50  0000 C CNN
-F 2 "" H 3950 4150 50  0000 C CNN
+F 2 "Pin_Headers:Pin_Header_Straight_1x05_Pitch2.54mm" H 3950 4150 50  0001 C CNN
 F 3 "" H 3950 4150 50  0000 C CNN
 	1    3950 4150
@@
 F 0 "P7" H 3950 6100 50  0000 C CNN
 F 1 "PROG_CON_2" V 4050 5800 50  0000 C CNN
-F 2 "" H 3950 5800 50  0000 C CNN
+F 2 "Pin_Headers:Pin_Header_Straight_1x05_Pitch2.54mm" H 3950 5800 50  0001 C CNN
 F 3 "" H 3950 5800 50  0000 C CNN
 	1    3950 5800
@@
 F 0 "P4" H 3950 3000 50  0000 C CNN
 F 1 "DEBUG_CON" V 4050 2850 50  0000 C CNN
-F 2 "" H 3950 2850 50  0000 C CNN
+F 2 "Pin_Headers:Pin_Header_Straight_1x02_Pitch2.54mm" H 3950 2850 50  0001 C CNN
 F 3 "" H 3950 2850 50  0000 C CNN
 	1    3950 2850
@@
 F 0 "P3" H 1650 1950 50  0000 C CNN
 F 1 "Battery_Charger_Output" V 1750 1800 50  0000 C CNN
-F 2 "" H 1650 1800 50  0000 C CNN
+F 2 "Pin_Headers:Pin_Header_Straight_1x02_Pitch2.54mm" H 1650 1800 50  0001 C CNN
 F 3 "" H 1650 1800 50  0000 C CNN
 	1    1650 1800
@@
 F 0 "P2" H 1100 3700 50  0000 C CNN
 F 1 "LIghts_Connector" V 1200 3150 50  0000 C CNN
-F 2 "" H 1100 3150 50  0000 C CNN
+F 2 "Pin_Headers:Pin_Header_Straight_1x10_Pitch2.54mm" H 1100 3150 50  0001 C CNN
 F 3 "" H 1100 3150 50  0000 C CNN
 	1    1100 3150
@@
 F 0 "R3" V 4530 1900 50  0000 C CNN
 F 1 "1k5" V 4450 1900 50  0000 C CNN
-F 2 "" V 4380 1900 50  0000 C CNN
+F 2 "Resistors_SMD:R_0805_HandSoldering" V 4380 1900 50  0001 C CNN
 F 3 "" H 4450 1900 50  0000 C CNN
 	1    4450 1900
@@
 F 0 "P15" H 1650 6200 50  0000 C CNN
 F 1 "light debug" V 1750 6050 50  0000 C CNN
-F 2 "" H 1650 6050 50  0000 C CNN
+F 2 "Pin_Headers:Pin_Header_Straight_1x02_Pitch2.54mm" H 1650 6050 50  0001 C CNN
 F 3 "" H 1650 6050 50  0000 C CNN
 	1    1650 6050
