File: 20-12-2016/EB_DRV/HALL_Filters.sch (KiCad schematic (older format))
At the start: 11 parts

Commit message: Added_footprints(not all)
Parts:
- C14, C15, C16, C17: footprint (none) -> Capacitors_SMD:C_0805_HandSoldering
- R12, R13, R14, R15, R16, R17, R18: footprint (none) -> Resistors_SMD:R_0805_HandSoldering
Changed lines of the file:
@@
 F 0 "R16" V 5180 3550 50  0000 C CNN
 F 1 "R" V 5100 3550 50  0000 C CNN
-F 2 "" V 5030 3550 50  0000 C CNN
+F 2 "Resistors_SMD:R_0805_HandSoldering" V 5030 3550 50  0001 C CNN
 F 3 "" H 5100 3550 50  0000 C CNN
 	1    5100 3550
@@
 F 0 "R17" V 5180 3750 50  0000 C CNN
 F 1 "R" V 5100 3750 50  0000 C CNN
-F 2 "" V 5030 3750 50  0000 C CNN
+F 2 "Resistors_SMD:R_0805_HandSoldering" V 5030 3750 50  0001 C CNN
 F 3 "" H 5100 3750 50  0000 C CNN
 	1    5100 3750
@@
 F 0 "R18" V 5180 3950 50  0000 C CNN
 F 1 "R" V 5100 3950 50  0000 C CNN
-F 2 "" V 5030 3950 50  0000 C CNN
+F 2 "Resistors_SMD:R_0805_HandSoldering" V 5030 3950 50  0001 C CNN
 F 3 "" H 5100 3950 50  0000 C CNN
 	1    5100 3950
@@
 F 0 "R15" V 4880 3050 50  0000 C CNN
 F 1 "R" V 4800 3050 50  0000 C CNN
-F 2 "" V 4730 3050 50  0000 C CNN
+F 2 "Resistors_SMD:R_0805_HandSoldering" V 4730 3050 50  0001 C CNN
 F 3 "" H 4800 3050 50  0000 C CNN
 	1    4800 3050
@@
 F 0 "R14" V 4680 3050 50  0000 C CNN
 F 1 "R" V 4600 3050 50  0000 C CNN
-F 2 "" V 4530 3050 50  0000 C CNN
+F 2 "Resistors_SMD:R_0805_HandSoldering" V 4530 3050 50  0001 C CNN
 F 3 "" H 4600 3050 50  0000 C CNN
 	1    4600 3050
@@
 F 0 "R13" V 4480 3050 50  0000 C CNN
 F 1 "R" V 4400 3050 50  0000 C CNN
-F 2 "" V 4330 3050 50  0000 C CNN
+F 2 "Resistors_SMD:R_0805_HandSoldering" V 4330 3050 50  0001 C CNN
 F 3 "" H 4400 3050 50  0000 C CNN
 	1    4400 3050
@@
 F 0 "R12" V 4280 3050 50  0000 C CNN
 F 1 "R" V 4200 3050 50  0000 C CNN
-F 2 "" V 4130 3050 50  0000 C CNN
+F 2 "Resistors_SMD:R_0805_HandSoldering" V 4130 3050 50  0001 C CNN
 F 3 "" H 4200 3050 50  0000 C CNN
 	1    4200 3050
@@
 F 0 "C14" H 5425 4400 50  0000 L CNN
 F 1 "C" H 5425 4200 50  0000 L CNN
-F 2 "" H 5438 4150 50  0000 C CNN
+F 2 "Capacitors_SMD:C_0805_HandSoldering" H 5438 4150 50  0001 C CNN
 F 3 "" H 5400 4300 50  0000 C CNN
 	1    5400 4300
@@
 F 0 "C15" H 5725 4400 50  0000 L CNN
 F 1 "C" H 5725 4200 50  0000 L CNN
-F 2 "" H 5738 4150 50  0000 C CNN
+F 2 "Capacitors_SMD:C_0805_HandSoldering" H 5738 4150 50  0001 C CNN
 F 3 "" H 5700 4300 50  0000 C CNN
 	1    5700 4300
@@
 F 0 "C16" H 6025 4400 50  0000 L CNN
 F 1 "C" H 6025 4200 50  0000 L CNN
-F 2 "" H 6038 4150 50  0000 C CNN
+F 2 "Capacitors_SMD:C_0805_HandSoldering" H 6038 4150 50  0001 C CNN
 F 3 "" H 6000 4300 50  0000 C CNN
 	1    6000 4300
@@
 F 0 "C17" H 6325 4400 50  0000 L CNN
 F 1 "C" H 6325 4200 50  0000 L CNN
-F 2 "" H 6338 4150 50  0000 C CNN
+F 2 "Capacitors_SMD:C_0805_HandSoldering" H 6338 4150 50  0001 C CNN
 F 3 "" H 6300 4300 50  0000 C CNN
 	1    6300 4300
