File: 20-12-2016/EB_DRV/Light_sensor.sch (KiCad schematic (older format))
At the start: 3 parts, among them P12 PhotoRes_CONN

Commit message: Added_footprints(not all)
Parts:
- P12: footprint (none) -> Pin_Headers:Pin_Header_Angled_1x02_Pitch2.54mm
Changed lines of the file:
@@
 U 1 1 5853D7F0
 P 6950 3600
+AR Path="/5853D7F0" Ref="P12"  Part="1"
+AR Path="/58516481/5853D7F0" Ref="P12"  Part="1"
 F 0 "P12" H 6950 3750 50  0000 C CNN
 F 1 "PhotoRes_CONN" V 7050 3600 50  0000 C CNN
-F 2 "" H 6950 3600 50  0000 C CNN
+F 2 "Pin_Headers:Pin_Header_Angled_1x02_Pitch2.54mm" H 6950 3600 50  0001 C CNN
 F 3 "" H 6950 3600 50  0000 C CNN
 	1    6950 3600
