File: 20-12-2016/EB_DRV/Lights.sch (KiCad schematic (older format))
At the start: 7 parts, among them P9 CONN_02X10, Q1 Q_NPN_BCE, Q2 Q_NPN_BCE

Commit message: Added_footprints(not all)
Parts:
- P9: footprint (none) -> Pin_Headers:Pin_Header_Straight_2x10_Pitch2.54mm
Changed lines of the file:
@@
 F 0 "P9" H 6000 3700 50  0000 C CNN
 F 1 "CONN_02X10" V 6000 3150 50  0000 C CNN
-F 2 "" H 6000 1950 50  0000 C CNN
+F 2 "Pin_Headers:Pin_Header_Straight_2x10_Pitch2.54mm" H 6000 1950 50  0001 C CNN
 F 3 "" H 6000 1950 50  0000 C CNN
 	1    6000 3150
