File: 20-12-2016/EB_DRV/MOSFET_PWR.sch (KiCad schematic (older format))
At the start: 15 parts, among them Q3 IRFS7530, Q4 IRFS7530, Q5 IRFS7530, Q6 IRFS7530, Q7 IRFS7530, Q8 IRFS7530

Commit message: Added_footprints(not all)
Parts:
- R56, R57, R58, R59, R60, R61, R62, R63, R64: footprint (none) -> Resistors_SMD:R_0805_HandSoldering
Changed lines of the file:
@@
 F 0 "R56" V 3280 2850 50  0000 C CNN
 F 1 "4R7" V 3200 2850 50  0000 C CNN
-F 2 "" V 3130 2850 50  0000 C CNN
+F 2 "Resistors_SMD:R_0805_HandSoldering" V 3130 2850 50  0001 C CNN
 F 3 "" H 3200 2850 50  0000 C CNN
 	1    3200 2850
@@
 F 0 "R59" V 5480 2800 50  0000 C CNN
 F 1 "4R7" V 5400 2800 50  0000 C CNN
-F 2 "" V 5330 2800 50  0000 C CNN
+F 2 "Resistors_SMD:R_0805_HandSoldering" V 5330 2800 50  0001 C CNN
 F 3 "" H 5400 2800 50  0000 C CNN
 	1    5400 2800
@@
 F 0 "R62" V 7630 2750 50  0000 C CNN
 F 1 "4R7" V 7550 2750 50  0000 C CNN
-F 2 "" V 7480 2750 50  0000 C CNN
+F 2 "Resistors_SMD:R_0805_HandSoldering" V 7480 2750 50  0001 C CNN
 F 3 "" H 7550 2750 50  0000 C CNN
 	1    7550 2750
@@
 F 0 "R57" V 3330 4250 50  0000 C CNN
 F 1 "4R7" V 3250 4250 50  0000 C CNN
-F 2 "" V 3180 4250 50  0000 C CNN
+F 2 "Resistors_SMD:R_0805_HandSoldering" V 3180 4250 50  0001 C CNN
 F 3 "" H 3250 4250 50  0000 C CNN
 	1    3250 4250
@@
 F 0 "R60" V 5530 4250 50  0000 C CNN
 F 1 "4R7" V 5450 4250 50  0000 C CNN
-F 2 "" V 5380 4250 50  0000 C CNN
+F 2 "Resistors_SMD:R_0805_HandSoldering" V 5380 4250 50  0001 C CNN
 F 3 "" H 5450 4250 50  0000 C CNN
 	1    5450 4250
@@
 F 0 "R63" V 7730 4250 50  0000 C CNN
 F 1 "4R7" V 7650 4250 50  0000 C CNN
-F 2 "" V 7580 4250 50  0000 C CNN
+F 2 "Resistors_SMD:R_0805_HandSoldering" V 7580 4250 50  0001 C CNN
 F 3 "" H 7650 4250 50  0000 C CNN
 	1    7650 4250
@@
 F 0 "R58" V 3580 4700 50  0000 C CNN
 F 1 "39k" V 3500 4700 50  0000 C CNN
-F 2 "" V 3430 4700 50  0000 C CNN
+F 2 "Resistors_SMD:R_0805_HandSoldering" V 3430 4700 50  0001 C CNN
 F 3 "" H 3500 4700 50  0000 C CNN
 	1    3500 4700
@@
 F 0 "R61" V 5730 4800 50  0000 C CNN
 F 1 "39k" V 5650 4800 50  0000 C CNN
-F 2 "" V 5580 4800 50  0000 C CNN
+F 2 "Resistors_SMD:R_0805_HandSoldering" V 5580 4800 50  0001 C CNN
 F 3 "" H 5650 4800 50  0000 C CNN
 	1    5650 4800
@@
 F 0 "R64" V 7930 4750 50  0000 C CNN
 F 1 "39k" V 7850 4750 50  0000 C CNN
-F 2 "" V 7780 4750 50  0000 C CNN
+F 2 "Resistors_SMD:R_0805_HandSoldering" V 7780 4750 50  0001 C CNN
 F 3 "" H 7850 4750 50  0000 C CNN
 	1    7850 4750
