File: 20-12-2016/EB_DRV/Mosfet_Driver.sch (KiCad schematic (older format))
At the start: 41 parts, among them U4 DRV8302

Commit message: Added_footprints(not all)
Parts:
- C29, C30, C31, C32, C33, C34, C35, C36, C37, C38, C39, C40, C41, C42, C43, C44, C45, C46: footprint (none) -> Capacitors_SMD:C_0805_HandSoldering
- R35, R36, R37, R38, R39, R40, R41, R42, R43, R44, R45, R46, R47, R48, R49, R50, R51, R52, R53, R54, R55: footprint (none) -> Resistors_SMD:R_0805_HandSoldering
Changed lines of the file:
@@
 F 0 "C35" H 6875 2000 50  0000 L CNN
 F 1 "0,015uF" H 6875 1800 50  0000 L CNN
-F 2 "" H 6888 1750 50  0000 C CNN
+F 2 "Capacitors_SMD:C_0805_HandSoldering" H 6888 1750 50  0001 C CNN
 F 3 "" H 6850 1900 50  0000 C CNN
 	1    6850 1900
@@
 F 0 "C40" V 7200 2600 50  0000 L CNN
 F 1 "0,1u" V 7200 2850 50  0000 L CNN
-F 2 "" H 7288 2600 50  0000 C CNN
+F 2 "Capacitors_SMD:C_0805_HandSoldering" H 7288 2600 50  0001 C CNN
 F 3 "" H 7250 2750 50  0000 C CNN
 	1    7250 2750
@@
 F 0 "C46" H 9775 3200 50  0000 L CNN
 F 1 "47uF" H 9775 3000 50  0000 L CNN
-F 2 "" H 9788 2950 50  0000 C CNN
+F 2 "Capacitors_SMD:C_0805_HandSoldering" H 9788 2950 50  0001 C CNN
 F 3 "" H 9750 3100 50  0000 C CNN
 	1    9750 3100
@@
 F 0 "R54" V 10280 3100 50  0000 C CNN
 F 1 "R" V 10200 3100 50  0000 C CNN
-F 2 "" V 10130 3100 50  0000 C CNN
+F 2 "Resistors_SMD:R_0805_HandSoldering" V 10130 3100 50  0001 C CNN
 F 3 "" H 10200 3100 50  0000 C CNN
 	1    10200 3100
@@
 F 0 "R55" V 10280 3500 50  0000 C CNN
 F 1 "R" V 10200 3500 50  0000 C CNN
-F 2 "" V 10130 3500 50  0000 C CNN
+F 2 "Resistors_SMD:R_0805_HandSoldering" V 10130 3500 50  0001 C CNN
 F 3 "" H 10200 3500 50  0000 C CNN
 	1    10200 3500
@@
 F 0 "C37" V 6950 3000 50  0000 L CNN
 F 1 "0,1u" V 6950 3250 50  0000 L CNN
-F 2 "" H 7038 3000 50  0000 C CNN
+F 2 "Capacitors_SMD:C_0805_HandSoldering" H 7038 3000 50  0001 C CNN
 F 3 "" H 7000 3150 50  0000 C CNN
 	1    7000 3150
@@
 F 0 "C38" V 6950 3500 50  0000 L CNN
 F 1 "0,1u" V 6950 3750 50  0000 L CNN
-F 2 "" H 7038 3500 50  0000 C CNN
+F 2 "Capacitors_SMD:C_0805_HandSoldering" H 7038 3500 50  0001 C CNN
 F 3 "" H 7000 3650 50  0000 C CNN
 	1    7000 3650
@@
 F 0 "C39" V 6950 4000 50  0000 L CNN
 F 1 "0,1u" V 6950 4250 50  0000 L CNN
-F 2 "" H 7038 4000 50  0000 C CNN
+F 2 "Capacitors_SMD:C_0805_HandSoldering" H 7038 4000 50  0001 C CNN
 F 3 "" H 7000 4150 50  0000 C CNN
 	1    7000 4150
@@
 F 0 "C32" V 4050 3500 50  0000 L CNN
 F 1 "0.022uF" V 4050 3750 50  0000 L CNN
-F 2 "" H 4138 3500 50  0000 C CNN
+F 2 "Capacitors_SMD:C_0805_HandSoldering" H 4138 3500 50  0001 C CNN
 F 3 "" H 4100 3650 50  0000 C CNN
 	1    4100 3650
@@
 F 0 "C36" H 6875 5300 50  0000 L CNN
 F 1 "0,1uF" H 6875 5100 50  0000 L CNN
-F 2 "" H 6888 5050 50  0000 C CNN
+F 2 "Capacitors_SMD:C_0805_HandSoldering" H 6888 5050 50  0001 C CNN
 F 3 "" H 6850 5200 50  0000 C CNN
 	1    6850 5200
@@
 F 0 "C41" H 7275 5300 50  0000 L CNN
 F 1 "4,7uF" H 7275 5100 50  0000 L CNN
-F 2 "" H 7288 5050 50  0000 C CNN
+F 2 "Capacitors_SMD:C_0805_HandSoldering" H 7288 5050 50  0001 C CNN
 F 3 "" H 7250 5200 50  0000 C CNN
 	1    7250 5200
@@
 F 0 "C42" H 7425 2000 50  0000 L CNN
 F 1 "0,1uF" H 7425 1800 50  0000 L CNN
-F 2 "" H 7438 1750 50  0000 C CNN
+F 2 "Capacitors_SMD:C_0805_HandSoldering" H 7438 1750 50  0001 C CNN
 F 3 "" H 7400 1900 50  0000 C CNN
 	1    7400 1900
@@
 F 0 "C43" H 7825 2000 50  0000 L CNN
 F 1 "4,7uF" H 7825 1800 50  0000 L CNN
-F 2 "" H 7838 1750 50  0000 C CNN
+F 2 "Capacitors_SMD:C_0805_HandSoldering" H 7838 1750 50  0001 C CNN
 F 3 "" H 7800 1900 50  0000 C CNN
 	1    7800 1900
@@
 F 0 "C30" H 3025 3900 50  0000 L CNN
 F 1 "2,2uF" H 3025 3700 50  0000 L CNN
-F 2 "" H 3038 3650 50  0000 C CNN
+F 2 "Capacitors_SMD:C_0805_HandSoldering" H 3038 3650 50  0001 C CNN
 F 3 "" H 3000 3800 50  0000 C CNN
 	1    3000 3800
@@
 F 0 "C29" H 1425 4900 50  0000 L CNN
 F 1 "1uF" H 1425 4700 50  0000 L CNN
-F 2 "" H 1438 4650 50  0000 C CNN
+F 2 "Capacitors_SMD:C_0805_HandSoldering" H 1438 4650 50  0001 C CNN
 F 3 "" H 1400 4800 50  0000 C CNN
 	1    1400 4800
@@
 F 0 "C34" H 4375 5400 50  0000 L CNN
 F 1 "1uF" H 4375 5200 50  0000 L CNN
-F 2 "" H 4388 5150 50  0000 C CNN
+F 2 "Capacitors_SMD:C_0805_HandSoldering" H 4388 5150 50  0001 C CNN
 F 3 "" H 4350 5300 50  0000 C CNN
 	1    4350 5300
@@
 F 0 "R42" V 5080 1550 50  0000 C CNN
 F 1 "205k" V 5000 1550 50  0000 C CNN
-F 2 "" V 4930 1550 50  0000 C CNN
+F 2 "Resistors_SMD:R_0805_HandSoldering" V 4930 1550 50  0001 C CNN
 F 3 "" H 5000 1550 50  0000 C CNN
 	1    5000 1550
@@
 F 0 "R38" V 4130 1250 50  0000 C CNN
 F 1 "16,2k" V 4050 1250 50  0000 C CNN
-F 2 "" V 3980 1250 50  0000 C CNN
+F 2 "Resistors_SMD:R_0805_HandSoldering" V 3980 1250 50  0001 C CNN
 F 3 "" H 4050 1250 50  0000 C CNN
 	1    4050 1250
@@
 F 0 "C31" H 4075 1700 50  0000 L CNN
 F 1 "6800pF" H 4075 1500 50  0000 L CNN
-F 2 "" H 4088 1450 50  0000 C CNN
+F 2 "Capacitors_SMD:C_0805_HandSoldering" H 4088 1450 50  0001 C CNN
 F 3 "" H 4050 1600 50  0000 C CNN
 	1    4050 1600
@@
 F 0 "C33" H 4375 1500 50  0000 L CNN
 F 1 "120pF" H 4375 1300 50  0000 L CNN
-F 2 "" H 4388 1250 50  0000 C CNN
+F 2 "Capacitors_SMD:C_0805_HandSoldering" H 4388 1250 50  0001 C CNN
 F 3 "" H 4350 1400 50  0000 C CNN
 	1    4350 1400
@@
 F 0 "R37" V 3630 2200 50  0000 C CNN
 F 1 "10k" V 3550 2200 50  0000 C CNN
-F 2 "" V 3480 2200 50  0000 C CNN
+F 2 "Resistors_SMD:R_0805_HandSoldering" V 3480 2200 50  0001 C CNN
 F 3 "" H 3550 2200 50  0000 C CNN
 	1    3550 2200
@@
 F 0 "R36" V 3630 1700 50  0000 C CNN
 F 1 "31,6k" V 3550 1700 50  0000 C CNN
-F 2 "" V 3480 1700 50  0000 C CNN
+F 2 "Resistors_SMD:R_0805_HandSoldering" V 3480 1700 50  0001 C CNN
 F 3 "" H 3550 1700 50  0000 C CNN
 	1    3550 1700
@@
 F 0 "R41" V 4380 2950 50  0000 C CNN
 F 1 "1" V 4300 2950 50  0000 C CNN
-F 2 "" V 4230 2950 50  0000 C CNN
+F 2 "Resistors_SMD:R_0805_HandSoldering" V 4230 2950 50  0001 C CNN
 F 3 "" H 4300 2950 50  0000 C CNN
 	1    4300 2950
@@
 F 0 "R40" V 4150 5050 50  0000 C CNN
 F 1 "R" V 4100 4850 50  0000 C CNN
-F 2 "" V 4030 4850 50  0000 C CNN
+F 2 "Resistors_SMD:R_0805_HandSoldering" V 4030 4850 50  0001 C CNN
 F 3 "" H 4100 4850 50  0000 C CNN
 	1    4100 4850
@@
 F 0 "R39" V 4050 4950 50  0000 C CNN
 F 1 "R" V 4100 4750 50  0000 C CNN
-F 2 "" V 4030 4750 50  0000 C CNN
+F 2 "Resistors_SMD:R_0805_HandSoldering" V 4030 4750 50  0001 C CNN
 F 3 "" H 4100 4750 50  0000 C CNN
 	1    4100 4750
@@
 F 0 "R43" V 6830 3050 50  0000 C CNN
 F 1 "1M" V 6750 3050 50  0000 C CNN
-F 2 "" V 6680 3050 50  0000 C CNN
+F 2 "Resistors_SMD:R_0805_HandSoldering" V 6680 3050 50  0001 C CNN
 F 3 "" H 6750 3050 50  0000 C CNN
 	1    6750 3050
@@
 F 0 "R35" V 3430 2200 50  0000 C CNN
 F 1 "10k" V 3350 2200 50  0000 C CNN
-F 2 "" V 3280 2200 50  0000 C CNN
+F 2 "Resistors_SMD:R_0805_HandSoldering" V 3280 2200 50  0001 C CNN
 F 3 "" H 3350 2200 50  0000 C CNN
 	1    3350 2200
@@
 F 0 "R44" V 8730 3350 50  0000 C CNN
 F 1 "39k" V 8650 3350 50  0000 C CNN
-F 2 "" V 8580 3350 50  0000 C CNN
+F 2 "Resistors_SMD:R_0805_HandSoldering" V 8580 3350 50  0001 C CNN
 F 3 "" H 8650 3350 50  0000 C CNN
 	1    8650 3350
@@
 F 0 "R45" V 8730 3500 50  0000 C CNN
 F 1 "2k2" V 8650 3500 50  0000 C CNN
-F 2 "" V 8580 3500 50  0000 C CNN
+F 2 "Resistors_SMD:R_0805_HandSoldering" V 8580 3500 50  0001 C CNN
 F 3 "" H 8650 3500 50  0000 C CNN
 	1    8650 3500
@@
 F 0 "R46" V 8730 3850 50  0000 C CNN
 F 1 "39k" V 8650 3850 50  0000 C CNN
-F 2 "" V 8580 3850 50  0000 C CNN
+F 2 "Resistors_SMD:R_0805_HandSoldering" V 8580 3850 50  0001 C CNN
 F 3 "" H 8650 3850 50  0000 C CNN
 	1    8650 3850
@@
 F 0 "R47" V 8730 4000 50  0000 C CNN
 F 1 "2k2" V 8650 4000 50  0000 C CNN
-F 2 "" V 8580 4000 50  0000 C CNN
+F 2 "Resistors_SMD:R_0805_HandSoldering" V 8580 4000 50  0001 C CNN
 F 3 "" H 8650 4000 50  0000 C CNN
 	1    8650 4000
@@
 F 0 "R48" V 8730 4350 50  0000 C CNN
 F 1 "39k" V 8650 4350 50  0000 C CNN
-F 2 "" V 8580 4350 50  0000 C CNN
+F 2 "Resistors_SMD:R_0805_HandSoldering" V 8580 4350 50  0001 C CNN
 F 3 "" H 8650 4350 50  0000 C CNN
 	1    8650 4350
@@
 F 0 "R49" V 8730 4500 50  0000 C CNN
 F 1 "2k2" V 8650 4500 50  0000 C CNN
-F 2 "" V 8580 4500 50  0000 C CNN
+F 2 "Resistors_SMD:R_0805_HandSoldering" V 8580 4500 50  0001 C CNN
 F 3 "" H 8650 4500 50  0000 C CNN
 	1    8650 4500
@@
 F 0 "C44" H 9025 4750 50  0000 L CNN
 F 1 "C" H 9025 4550 50  0000 L CNN
-F 2 "" H 9038 4500 50  0000 C CNN
+F 2 "Capacitors_SMD:C_0805_HandSoldering" H 9038 4500 50  0001 C CNN
 F 3 "" H 9000 4650 50  0000 C CNN
 	1    9000 4650
@@
 F 0 "C45" H 9025 4950 50  0000 L CNN
 F 1 "C" H 9025 4750 50  0000 L CNN
-F 2 "" H 9038 4700 50  0000 C CNN
+F 2 "Capacitors_SMD:C_0805_HandSoldering" H 9038 4700 50  0001 C CNN
 F 3 "" H 9000 4850 50  0000 C CNN
 	1    9000 4850
@@
 F 0 "R50" V 9880 5000 50  0000 C CNN
 F 1 "R" V 9800 5000 50  0000 C CNN
-F 2 "" V 9730 5000 50  0000 C CNN
+F 2 "Resistors_SMD:R_0805_HandSoldering" V 9730 5000 50  0001 C CNN
 F 3 "" H 9800 5000 50  0000 C CNN
 	1    9800 5000
@@
 F 0 "R51" V 9880 5150 50  0000 C CNN
 F 1 "R" V 9800 5150 50  0000 C CNN
-F 2 "" V 9730 5150 50  0000 C CNN
+F 2 "Resistors_SMD:R_0805_HandSoldering" V 9730 5150 50  0001 C CNN
 F 3 "" H 9800 5150 50  0000 C CNN
 	1    9800 5150
@@
 F 0 "R52" V 9880 5400 50  0000 C CNN
 F 1 "R" V 9800 5400 50  0000 C CNN
-F 2 "" V 9730 5400 50  0000 C CNN
+F 2 "Resistors_SMD:R_0805_HandSoldering" V 9730 5400 50  0001 C CNN
 F 3 "" H 9800 5400 50  0000 C CNN
 	1    9800 5400
@@
 F 0 "R53" V 9880 5550 50  0000 C CNN
 F 1 "R" V 9800 5550 50  0000 C CNN
-F 2 "" V 9730 5550 50  0000 C CNN
+F 2 "Resistors_SMD:R_0805_HandSoldering" V 9730 5550 50  0001 C CNN
 F 3 "" H 9800 5550 50  0000 C CNN
 	1    9800 5550
