File: 20-12-2016/EB_DRV/PCB_Temp.sch (KiCad schematic (older format))
At the start: 3 parts

Commit message: Added_footprints(not all)
Parts:
- C47: footprint (none) -> Capacitors_SMD:C_0805_HandSoldering
- R67, R68: footprint (none) -> Resistors_SMD:R_0805_HandSoldering
Changed lines of the file:
@@
 F 0 "R67" V 5180 2700 50  0000 C CNN
 F 1 "1k" V 5100 2700 50  0000 C CNN
-F 2 "" V 5030 2700 50  0000 C CNN
+F 2 "Resistors_SMD:R_0805_HandSoldering" V 5030 2700 50  0001 C CNN
 F 3 "" H 5100 2700 50  0000 C CNN
 	1    5100 2700
@@
 F 0 "R68" V 5180 3350 50  0000 C CNN
 F 1 "NTC 10k" V 5000 3350 50  0000 C CNN
-F 2 "" V 5030 3350 50  0000 C CNN
+F 2 "Resistors_SMD:R_0805_HandSoldering" V 5030 3350 50  0001 C CNN
 F 3 "" H 5100 3350 50  0000 C CNN
 	1    5100 3350
@@
 F 0 "C47" H 5575 3450 50  0000 L CNN
 F 1 "C" H 5575 3250 50  0000 L CNN
-F 2 "" H 5588 3200 50  0000 C CNN
+F 2 "Capacitors_SMD:C_0805_HandSoldering" H 5588 3200 50  0001 C CNN
 F 3 "" H 5550 3350 50  0000 C CNN
 	1    5550 3350
