File: 20-12-2016/EB_DRV/PWR_MNGR.sch (KiCad schematic (older format))
At the start: 13 parts, among them U6 LR12K4-G, U7 LR12K4-G

Commit message: Added_footprints(not all)
Parts:
- C48, C49, C50, C51: footprint (none) -> Capacitors_SMD:C_0805_HandSoldering
- R69, R70, R71, R72, R74, R75, R76: footprint (none) -> Resistors_SMD:R_0805_HandSoldering
Changed lines of the file:
@@
 F 0 "C48" H 3325 2900 50  0000 L CNN
 F 1 "CP" H 3325 2700 50  0000 L CNN
-F 2 "" H 3338 2650 50  0000 C CNN
+F 2 "Capacitors_SMD:C_0805_HandSoldering" H 3338 2650 50  0001 C CNN
 F 3 "" H 3300 2800 50  0000 C CNN
 	1    3300 2800
@@
 F 0 "C49" H 5125 2850 50  0000 L CNN
 F 1 "100n" H 5125 2650 50  0000 L CNN
-F 2 "" H 5138 2600 50  0000 C CNN
+F 2 "Capacitors_SMD:C_0805_HandSoldering" H 5138 2600 50  0001 C CNN
 F 3 "" H 5100 2750 50  0000 C CNN
 	1    5100 2750
@@
 F 0 "R70" V 4780 2750 50  0000 C CNN
 F 1 "6k04" V 4700 2750 50  0000 C CNN
-F 2 "" V 4630 2750 50  0000 C CNN
+F 2 "Resistors_SMD:R_0805_HandSoldering" V 4630 2750 50  0001 C CNN
 F 3 "" H 4700 2750 50  0000 C CNN
 	1    4700 2750
@@
 F 0 "R69" V 4130 3250 50  0000 C CNN
 F 1 "18k2" V 4050 3250 50  0000 C CNN
-F 2 "" V 3980 3250 50  0000 C CNN
+F 2 "Resistors_SMD:R_0805_HandSoldering" V 3980 3250 50  0001 C CNN
 F 3 "" H 4050 3250 50  0000 C CNN
 	1    4050 3250
@@
 F 0 "R72" V 8830 2700 50  0000 C CNN
 F 1 "6k04" V 8750 2700 50  0000 C CNN
-F 2 "" V 8680 2700 50  0000 C CNN
+F 2 "Resistors_SMD:R_0805_HandSoldering" V 8680 2700 50  0001 C CNN
 F 3 "" H 8750 2700 50  0000 C CNN
 	1    8750 2700
@@
 F 0 "R71" V 8080 3300 50  0000 C CNN
 F 1 "10k1" V 8000 3300 50  0000 C CNN
-F 2 "" V 7930 3300 50  0000 C CNN
+F 2 "Resistors_SMD:R_0805_HandSoldering" V 7930 3300 50  0001 C CNN
 F 3 "" H 8000 3300 50  0000 C CNN
 	1    8000 3300
@@
 F 0 "C50" H 7225 2850 50  0000 L CNN
 F 1 "CP" H 7225 2650 50  0000 L CNN
-F 2 "" H 7238 2600 50  0000 C CNN
+F 2 "Capacitors_SMD:C_0805_HandSoldering" H 7238 2600 50  0001 C CNN
 F 3 "" H 7200 2750 50  0000 C CNN
 	1    7200 2750
@@
 F 0 "C51" H 9225 2800 50  0000 L CNN
 F 1 "CP" H 9225 2600 50  0000 L CNN
-F 2 "" H 9238 2550 50  0000 C CNN
+F 2 "Capacitors_SMD:C_0805_HandSoldering" H 9238 2550 50  0001 C CNN
 F 3 "" H 9200 2700 50  0000 C CNN
 	1    9200 2700
@@
 F 0 "R75" V 4830 5600 50  0000 C CNN
 F 1 "0R" V 4750 5600 50  0000 C CNN
-F 2 "" V 4680 5600 50  0000 C CNN
+F 2 "Resistors_SMD:R_0805_HandSoldering" V 4680 5600 50  0001 C CNN
 F 3 "" H 4750 5600 50  0000 C CNN
 	1    4750 5600
@@
 F 0 "R76" V 5180 5250 50  0000 C CNN
 F 1 "0R" V 5100 5250 50  0000 C CNN
-F 2 "" V 5030 5250 50  0000 C CNN
+F 2 "Resistors_SMD:R_0805_HandSoldering" V 5030 5250 50  0001 C CNN
 F 3 "" H 5100 5250 50  0000 C CNN
 	1    5100 5250
@@
 F 0 "R74" V 4480 5250 50  0000 C CNN
 F 1 "0R" V 4400 5250 50  0000 C CNN
-F 2 "" V 4330 5250 50  0000 C CNN
+F 2 "Resistors_SMD:R_0805_HandSoldering" V 4330 5250 50  0001 C CNN
 F 3 "" H 4400 5250 50  0000 C CNN
 	1    4400 5250
